Commit message: fourpm

File: src/loki_bringup/urdf/Full_Assembly_URDF_Combined.urdf (robot description, URDF)
Before this commit: robot Full_Assembly_URDF_Combined, 13 links, 12 joints
Links:
- link BottomRudder1_Link: geometry collision mesh filename=package://loki_bringup/meshes/BottomRudder1_Link.STL; visual mesh filename=package://loki_bringup/meshes/BottomRudder1_Link.STL
- link BottomRudder2_Joint: geometry collision mesh filename=package://loki_bringup/meshes/BottomRudder2_Joint.STL; visual mesh filename=package://loki_bringup/meshes/BottomRudder2_Joint.STL
- link Elevator1_Link: geometry collision mesh filename=package://loki_bringup/meshes/Elevator1_Link.STL; visual mesh filename=package://loki_bringup/meshes/Elevator1_Link.STL
- link Elevator2_Link: geometry collision mesh filename=package://loki_bringup/meshes/Elevator2_Link.STL; visual mesh filename=package://loki_bringup/meshes/Elevator2_Link.STL
- link Thruster1_Link: geometry collision mesh filename=package://loki_bringup/meshes/Thruster1_Link.STL; visual mesh filename=package://loki_bringup/meshes/Thruster1_Link.STL
- link Thruster2_Link: geometry collision mesh filename=package://loki_bringup/meshes/Thruster2_Link.STL; visual mesh filename=package://loki_bringup/meshes/Thruster2_Link.STL
- link TopRudder1_Link: geometry collision mesh filename=package://loki_bringup/meshes/TopRudder1_Link.STL; visual mesh filename=package://loki_bringup/meshes/TopRudder1_Link.STL
- link TopRudder2_Link: geometry collision mesh filename=package://loki_bringup/meshes/TopRudder2_Link.STL; visual mesh filename=package://loki_bringup/meshes/TopRudder2_Link.STL
- link base_link: geometry collision mesh filename=package://loki_bringup/meshes/base_link.STL; visual mesh filename=package://loki_bringup/meshes/base_link.STL
- link dvl_link: geometry collision mesh filename=package://loki_bringup/meshes/DVL_Link.STL; visual mesh filename=package://loki_bringup/meshes/DVL_Link.STL
